File: HDW_BUSINESS_CARD.kicad_pcb (KiCad board)
At the start: 2 copper layers, 89.4 x 51 mm, 10 parts, among them U1 NT3H1101

Commit message: now I actualy set up net classes for the coil properly
Routing:
- net Net-(D1-K): track 7.49 -> 2.00 mm, vias 1 -> 0
- net Net-(U1-LB): track 2.91 -> 6.15 mm, vias 0 -> 1
- net Net-(U1-LA): track 2.61 -> 4.17 mm
Changed lines of the file:
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@@
 	)
 	(gr_line
+		(start 71.27 83.27)
+		(end 73.51 84.45)
+		(stroke
+			(width 0.3)
+			(type default)
+		)
+		(layer "F.Cu")
+		(net 2)
+	)
+	(gr_line
 		(start 89.98 62.244443)
 		(end 74.78 53.468719)
@@
 		)
 		(layer "B.Cu")
-		(net 1)
+		(net 2)
 	)
 	(gr_line
@@
 		)
 		(layer "B.Cu")
-		(net 1)
+		(net 2)
 	)
 	(gr_line
@@
 		)
 		(layer "B.Cu")
-		(net 1)
+		(net 2)
 	)
 	(gr_line
@@
 		)
 		(layer "B.Cu")
-		(net 1)
+		(net 2)
 	)
 	(gr_line
@@
 		)
 		(layer "B.Cu")
-		(net 1)
+		(net 2)
 	)
 	(gr_line
@@
 		)
 		(layer "B.Cu")
-		(net 1)
+		(net 2)
 	)
 	(gr_line
@@
 		)
 		(layer "B.Cu")
-		(net 1)
+		(net 2)
 	)
 	(gr_line
@@
 		)
 		(layer "B.Cu")
-		(net 1)
+		(net 2)
 	)
 	(gr_line
@@
 		)
 		(layer "B.Cu")
-		(net 1)
+		(net 2)
 	)
 	(gr_line
@@
 		)
 		(layer "B.Cu")
-		(net 1)
+		(net 2)
 	)
 	(gr_line
@@
 		)
 		(layer "B.Cu")
-		(net 1)
+		(net 2)
 	)
 	(gr_line
@@
 		)
 		(layer "B.Cu")
-		(net 1)
+		(net 2)
 	)
 	(gr_line
@@
 		)
 		(layer "B.Cu")
-		(net 1)
+		(net 2)
 	)
 	(gr_line
@@
 		)
 		(layer "B.Cu")
-		(net 1)
+		(net 2)
 	)
 	(gr_line
@@
 		)
 		(layer "B.Cu")
-		(net 1)
+		(net 2)
 	)
 	(gr_line
@@
 		)
 		(layer "B.Cu")
-		(net 1)
+		(net 2)
 	)
 	(gr_line
@@
 		)
 		(layer "B.Cu")
-		(net 1)
+		(net 2)
 	)
 	(gr_line
@@
 		)
 		(layer "B.Cu")
-		(net 1)
+		(net 2)
 	)
 	(gr_line
@@
 		)
 		(layer "B.Cu")
-		(net 1)
+		(net 3)
 	)
 	(gr_line
@@
 		)
 		(layer "B.Cu")
-		(net 1)
+		(net 2)
 	)
 	(gr_line
@@
 		)
 		(layer "B.Cu")
-		(net 1)
+		(net 2)
 	)
 	(gr_line
@@
 		)
 		(layer "B.Cu")
-		(net 1)
+		(net 2)
 	)
 	(gr_line
@@
 		)
 		(layer "B.Cu")
-		(net 1)
+		(net 2)
 	)
 	(gr_line
@@
 		)
 		(layer "B.Cu")
-		(net 1)
+		(net 2)
 	)
 	(gr_line
@@
 		)
 		(layer "B.Cu")
-		(net 1)
+		(net 2)
 	)
 	(gr_line
@@
 		)
 		(layer "B.Cu")
-		(net 1)
+		(net 2)
 	)
 	(gr_line
@@
 		)
 		(layer "B.Cu")
-		(net 1)
+		(net 2)
 	)
 	(gr_line
@@
 		)
 		(layer "B.Cu")
-		(net 1)
+		(net 2)
 	)
 	(gr_line
@@
 		)
 		(layer "B.Cu")
-		(net 1)
+		(net 2)
 	)
 	(gr_line
@@
 		)
 		(layer "B.Cu")
-		(net 1)
+		(net 2)
 	)
 	(gr_line
@@
 		)
 		(layer "B.Cu")
-		(net 1)
+		(net 2)
 	)
 	(gr_line
@@
 		)
 		(layer "B.Cu")
-		(net 1)
+		(net 2)
 	)
 	(gr_line
@@
 		)
 		(layer "B.Cu")
-		(net 1)
+		(net 2)
 	)
 	(gr_line
@@
 		)
 		(layer "B.Cu")
-		(net 1)
+		(net 2)
 	)
 	(gr_line
@@
 		)
 		(layer "B.Cu")
-		(net 1)
+		(net 2)
 	)
 	(gr_line
@@
 		)
 		(layer "B.Cu")
-		(net 1)
+		(net 2)
 	)
 	(gr_line
@@
 		)
 		(layer "B.Cu")
-		(net 1)
+		(net 2)
 	)
 	(gr_line
@@
 		)
 		(layer "B.Cu")
-		(net 1)
+		(net 2)
 	)
 	(gr_line
@@
 		)
 		(layer "B.Cu")
-		(net 1)
+		(net 2)
 	)
 	(gr_line
@@
 		)
 		(layer "B.Cu")
-		(net 1)
+		(net 2)
 	)
 	(gr_line
@@
 		)
 		(layer "B.Cu")
-		(net 1)
+		(net 2)
 	)
 	(gr_line
@@
 		)
 		(layer "B.Cu")
-		(net 1)
+		(net 2)
 	)
 	(gr_line
@@
 		)
 		(layer "B.Cu")
-		(net 1)
+		(net 2)
 	)
 	(gr_line
@@
 	)
 	(segment
-		(start 73.54 85.19)
-		(end 73.55 85.2)
-		(width 0.25)
-		(layer "F.Cu")
+		(start 68.4075 91.9)
+		(end 68.32 91.8125)
+		(width 0.3)
+		(layer "B.Cu")
 		(net 1)
 	)
 	(segment
-		(start 73.51 84.45)
-		(end 73.51 86)
+		(start 70.28 91.9)
+		(end 68.4075 91.9)
 		(width 0.3)
-		(layer "F.Cu")
+		(layer "B.Cu")
 		(net 1)
 	)
 	(segment
-		(start 70.9 89.2)
-		(end 70.9 87.8)
+		(start 73.54 85.19)
+		(end 73.55 85.2)
 		(width 0.25)
 		(layer "F.Cu")
-		(net 1)
+		(net 2)
 	)
 	(segment
 		(start 73.51 84.45)
-		(end 71.27 83.27)
+		(end 73.51 86)
 		(width 0.3)
 		(layer "F.Cu")
-		(net 1)
-	)
-	(via
-		(at 70.9 89.2)
-		(size 0.35)
-		(drill 0.3)
-		(layers "F.Cu" "B.Cu")
-		(free yes)
-		(net 1)
-	)
-	(segment
-		(start 68.4075 91.9)
-		(end 68.32 91.8125)
-		(width 0.3)
-		(layer "B.Cu")
-		(net 1)
-	)
-	(segment
-		(start 70.28 91.9)
-		(end 68.4075 91.9)
-		(width 0.3)
-		(layer "B.Cu")
-		(net 1)
+		(net 2)
 	)
 	(via
@@
 	)
 	(segment
+		(start 70.9 89.2)
+		(end 70.9 87.8)
+		(width 0.25)
+		(layer "F.Cu")
+		(net 3)
+	)
+	(via
+		(at 70.9 89.2)
+		(size 0.35)
+		(drill 0.3)
+		(layers "F.Cu" "B.Cu")
+		(free yes)
+		(net 3)
+	)
+	(segment
 		(start 75.2625 91.47)
 		(end 73.653174 91.47)
 		(width 0.3)
 		(layer "B.Cu")
+		(net 3)
+	)
+	(segment
+		(start 73.175 91.985)
+		(end 73.175 90.675)
+		(width 0.3)
+		(layer "B.Cu")
+		(net 3)
+	)
+	(segment
+		(start 73.175 90.675)
+		(end 72.8 90.3)
+		(width 0.3)
+		(layer "B.Cu")

Commit message: sending off to PCBWay for first order
Parts:
- moved D1 9.49 mm to (77.6, 94.8)
- moved U1 2.49 mm to (74.8, 94.6)
- moved R1 2.36 mm to (72.1, 95.4)
- moved C1 2.30 mm to (72.0, 93.8)
- moved C2 1.11 mm to (74.8, 92.1), turned to 0 degrees
Connections:
- C1 pad 1: Net-(U1-VOUT) -> Net-(U1-VCC)
- R1 pad 1: Net-(U1-VOUT) -> Net-(U1-VCC)
- U1 pad 2: Net-(U1-VOUT) -> Net-(D1-K)
- U1 pad 6: Net-(D1-K) -> Net-(U1-VCC)
- U1 pad 7: Net-(U1-VOUT) -> Net-(U1-VCC)
Routing:
- net Net-(D1-K): track 2.00 -> 16.6 mm
- net Net-(U1-VOUT): track 8.06 -> 0.00 mm
- net Net-(D1-A): track 2.06 -> 6.72 mm
- net Net-(U1-VCC): track 0.00 -> 4.08 mm
- net Net-(U1-LA): track 4.17 -> 6.22 mm
- net Net-(U1-LB): track 6.15 -> 4.72 mm
Other:
- board text added: "+1 647-518-4574"
- board text removed: "+1 647-538-XXXX"

Commit message: added mounting holes in corners
Parts:
- added REF**: MountingHole_2.7mm_M2.5_Pad_Via, MountingHole:MountingHole_2.7mm_M2.5_Pad_Via, F.Cu at (54.0, 54.0)
- added REF**: MountingHole_2.7mm_M2.5_Pad_Via, MountingHole:MountingHole_2.7mm_M2.5_Pad_Via, F.Cu at (137.0, 54.0)
- added REF**: MountingHole_2.7mm_M2.5_Pad_Via, MountingHole:MountingHole_2.7mm_M2.5_Pad_Via, F.Cu at (137.0, 98.6)
- added REF**: MountingHole_2.7mm_M2.5_Pad_Via, MountingHole:MountingHole_2.7mm_M2.5_Pad_Via, F.Cu at (54.0, 98.6)
