File: HDW_BUSINESS_CARD.kicad_pcb (KiCad board)
At the start: 2 copper layers, 89.4 x 51 mm, 14 parts, among them U1 NT3H1101

Commit message: removed C2
Parts:
- removed C2: 440nF, Capacitor_SMD:C_0603_1608Metric_Pad1.08x0.95mm_HandSolder
Routing:
- net Net-(U1-LB): track 4.72 -> 3.84 mm
